File: electronics/actuator/actuator.kicad_pcb (KiCad board)
At the start: 2 copper layers, 52.5 x 55 mm, 34 parts, among them J1 MOTOR_OUT, J2 PWR_IN, J3 Pinouts, J4 Pinouts, Q1 NTMFS4935NT1G, Q2 NTMFS4935NT1G, Q3 NTMFS4935NT1G, Q4 NTMFS4935NT1G, Q5 NTMFS4935NT1G, Q6 NTMFS4935NT1G, U1 drv8323rs

Commit message: Updated board.
Parts:
- C1, C2, C3, C7, C8: footprint Capacitor_SMD:C_0603_1608Metric -> Capacitor_SMD:C_1206_3216Metric
- C10, C9: footprint Capacitor_SMD:C_0603_1608Metric -> Capacitor_SMD:CP_Elec_6.3x5.4
- L1: footprint Inductor_SMD:L_1210_3225Metric -> Inductor_THT:L_Radial_D7.8mm_P5.00mm_Fastron_07HCP
- R2: footprint Resistor_SMD:R_0603_1608Metric_Pad1.05x0.95mm_HandSolder -> Resistor_SMD:R_0402_1005Metric
- R6, R7, R8: footprint Resistor_SMD:R_1210_3225Metric -> Resistor_SMD:R_2512_6332Metric
- moved C10 7.23 mm to (120.6, 68.6)
- moved C9 2.81 mm to (120.6, 61.1)
- moved R7 1.40 mm to (137.8, 83.0)
- moved R8 1.40 mm to (161.5, 83.0)
- moved C8 1.30 mm to (135.5, 56.0)
- moved L1 1.14 mm to (138.7, 55.4)
- moved C7 1.03 mm to (135.5, 60.8)
- moved C2 0.97 mm to (144.9, 83.2)
- moved R6 0.51 mm to (125.6, 82.9)
- moved R2 0.35 mm to (130.6, 62.6)
Routing:
- net VAA: track 43.7 -> 47.1 mm
- net SNA: track 61.8 -> 64.3 mm, vias 28 -> 22
- net GLB: track 11.9 -> 13.8 mm
- net SPA: track 14.7 -> 16.3 mm
- net SPB: track 10.3 -> 10.9 mm
- net GHA: track 28.8 -> 28.2 mm
