File: electronics/actuator/actuator.sch (KiCad schematic (older format))
At the start: 29 parts, among them J1 Screw_Terminal_01x03, Q1 NTMFS4935NT1G, Q2 NTMFS4935NT1G, Q3 NTMFS4935NT1G, Q4 NTMFS4935NT1G, Q5 NTMFS4935NT1G, Q6 NTMFS4935NT1G, U1 drv8323rs

Commit message: Added footprints.
Parts:
- removed C6, C7, C8: C_Small, symbol Device:C_Small
- 27uH1: renamed from L1; footprint (none) -> Inductor_SMD:L_1210_3225Metric
- C1, C5: value C_Small -> 0.1uF; footprint (none) -> Capacitor_SMD:C_0603_1608Metric
- C2: value C_Small -> 47uF; footprint (none) -> Capacitor_SMD:C_0603_1608Metric
- C3, C4: value C_Small -> 1uF; footprint (none) -> Capacitor_SMD:C_0603_1608Metric
- C6: renamed from C9; footprint (none) -> Capacitor_SMD:C_0603_1608Metric
- C7: renamed from C10; value C_Small -> 10uF; footprint (none) -> Capacitor_SMD:C_0603_1608Metric
- C8: renamed from C11; value C_Small -> 10uF; footprint (none) -> Capacitor_SMD:C_0603_1608Metric
- D1: footprint (none) -> Diode_SMD:D_SOD-123F
- J1: footprint (none) -> TerminalBlock_4Ucon:TerminalBlock_4Ucon_1x03_P3.50mm_Horizontal
- Q1, Q2, Q3, Q4, Q5, Q6: footprint Package_DirectFET:DirectFET_SH -> Package_DFN_QFN:TDFN-8-1EP_3x2mm_P0.5mm_EP1.80x1.65mm_ThermalVias
- R1: value R_Small -> 28k; footprint (none) -> Resistor_SMD:R_0603_1608Metric_Pad1.05x0.95mm_HandSolder
- R2: renamed from R5; value R_Small -> 8.45k; footprint (none) -> Resistor_SMD:R_0603_1608Metric_Pad1.05x0.95mm_HandSolder
- R3: renamed from R6; value R_Small -> 100k; footprint (none) -> Resistor_SMD:R_0603_1608Metric_Pad1.05x0.95mm_HandSolder
- R4: renamed from R7; value R_Small -> 10k; footprint (none) -> Resistor_SMD:R_0603_1608Metric_Pad1.05x0.95mm_HandSolder
- R5: renamed from R8; value R_Small -> 10k; footprint (none) -> Resistor_SMD:R_0603_1608Metric_Pad1.05x0.95mm_HandSolder
- R6: renamed from R2; value R -> 1m; footprint (none) -> Resistor_SMD:R_1210_3225Metric
- R7: renamed from R3; value R -> 1m; footprint (none) -> Resistor_SMD:R_1210_3225Metric
- R8: renamed from R4; value R -> 1m; footprint (none) -> Resistor_SMD:R_1210_3225Metric
- U1: footprint (none) -> Package_DFN_QFN:Texas_S-PVQFN-N48_EP5.15x5.15mm_ThermalVias; symbol custom_drv:drv8323rs -> actuator-rescue:drv8323rs-custom_drv
Connections:
- wire segments 140 -> 136

Commit message: Added SO-FL-8 footprint.
Parts:
- Q1, Q2, Q3, Q4, Q5, Q6: footprint Package_DFN_QFN:TDFN-8-1EP_3x2mm_P0.5mm_EP1.80x1.65mm_ThermalVias -> actuator:SO-FL-8
Changed lines of the file:
@@
 F 0 "Q1" H 5706 3396 50  0000 L CNN
 F 1 "NTMFS4935NT1G" H 5706 3305 50  0000 L CNN
-F 2 "Package_DFN_QFN:TDFN-8-1EP_3x2mm_P0.5mm_EP1.80x1.65mm_ThermalVias" H 5500 3350 50  0001 C CIN
+F 2 "actuator:SO-FL-8" H 5500 3350 50  0001 C CIN
 F 3 "https://www.infineon.com/dgdl/irf6665pbf.pdf?fileId=5546d462533600a4015355ec8dcb1a62" H 5500 3350 50  0001 L CNN
 	1    5500 3350
@@
 F 0 "Q3" H 6906 3396 50  0000 L CNN
 F 1 "NTMFS4935NT1G" H 6906 3305 50  0000 L CNN
-F 2 "Package_DFN_QFN:TDFN-8-1EP_3x2mm_P0.5mm_EP1.80x1.65mm_ThermalVias" H 6700 3350 50  0001 C CIN
+F 2 "actuator:SO-FL-8" H 6700 3350 50  0001 C CIN
 F 3 "https://www.infineon.com/dgdl/irf6665pbf.pdf?fileId=5546d462533600a4015355ec8dcb1a62" H 6700 3350 50  0001 L CNN
 	1    6700 3350
@@
 F 0 "Q5" H 8106 3396 50  0000 L CNN
 F 1 "NTMFS4935NT1G" H 8106 3305 50  0000 L CNN
-F 2 "Package_DFN_QFN:TDFN-8-1EP_3x2mm_P0.5mm_EP1.80x1.65mm_ThermalVias" H 7900 3350 50  0001 C CIN
+F 2 "actuator:SO-FL-8" H 7900 3350 50  0001 C CIN
 F 3 "https://www.infineon.com/dgdl/irf6665pbf.pdf?fileId=5546d462533600a4015355ec8dcb1a62" H 7900 3350 50  0001 L CNN
 	1    7900 3350
@@
 F 0 "Q2" H 5706 4096 50  0000 L CNN
 F 1 "NTMFS4935NT1G" H 5706 4005 50  0000 L CNN
-F 2 "Package_DFN_QFN:TDFN-8-1EP_3x2mm_P0.5mm_EP1.80x1.65mm_ThermalVias" H 5500 4050 50  0001 C CIN
+F 2 "actuator:SO-FL-8" H 5500 4050 50  0001 C CIN
 F 3 "https://www.infineon.com/dgdl/irf6665pbf.pdf?fileId=5546d462533600a4015355ec8dcb1a62" H 5500 4050 50  0001 L CNN
 	1    5500 4050
@@
 F 0 "Q4" H 6906 4096 50  0000 L CNN
 F 1 "NTMFS4935NT1G" H 6906 4005 50  0000 L CNN
-F 2 "Package_DFN_QFN:TDFN-8-1EP_3x2mm_P0.5mm_EP1.80x1.65mm_ThermalVias" H 6700 4050 50  0001 C CIN
+F 2 "actuator:SO-FL-8" H 6700 4050 50  0001 C CIN
 F 3 "https://www.infineon.com/dgdl/irf6665pbf.pdf?fileId=5546d462533600a4015355ec8dcb1a62" H 6700 4050 50  0001 L CNN
 	1    6700 4050
@@
 F 0 "Q6" H 8106 4096 50  0000 L CNN
 F 1 "NTMFS4935NT1G" H 8106 4005 50  0000 L CNN
-F 2 "Package_DFN_QFN:TDFN-8-1EP_3x2mm_P0.5mm_EP1.80x1.65mm_ThermalVias" H 7900 4050 50  0001 C CIN
+F 2 "actuator:SO-FL-8" H 7900 4050 50  0001 C CIN
 F 3 "https://www.infineon.com/dgdl/irf6665pbf.pdf?fileId=5546d462533600a4015355ec8dcb1a62" H 7900 4050 50  0001 L CNN
 	1    7900 4050

Commit message: Added a bunch of stuff and initial layout.
Parts:
- added C1, C2, C3: 10uF, Capacitor_SMD:C_0603_1608Metric, symbol Device:C_Small
- added C10, C9: 10uF, Capacitor_SMD:C_0603_1608Metric, symbol Device:CP_Small
- added J2: PWR_IN, connectors:PhoenixContact_GMSTBA_2,5_2-G-7,62_1x02_P7.62mm_Horizontal, symbol Connector:Conn_01x02_Female
- added J3, J4: Pinouts, Connector_PinSocket_2.54mm:PinSocket_1x08_P2.54mm_Vertical, symbol Connector:Conn_01x08_Female
- J1: value Screw_Terminal_01x03 -> MOTOR_OUT; footprint TerminalBlock_4Ucon:TerminalBlock_4Ucon_1x03_P3.50mm_Horizontal -> connectors:PhoenixContact_GMSTBA_2,5_3-G-7,62_1x03_P7.62mm_Horizontal
- renumbered C4 to C_DVDD1, C3 to C_SW1, C2 to C_VCP1, C1 to C_VM1
Connections:
- net DVDD: now also J3.7 (Pin_7)
- net ENABLE: now also J3.8 (Pin_8)
- net GND: now also C1.2, C10.2, C2.2, C3.2, C9.2, J2.1 (Pin_1)
- net INHA: now also J3.6 (Pin_6)
- net INHB: now also J3.4 (Pin_4)
- net INHC: now also J3.2 (Pin_2)
- net INLA: now also J3.5 (Pin_5)
- net INLB: now also J3.3 (Pin_3)
- net INLC: now also J3.1 (Pin_1)
- net SCLK: now also J4.2 (Pin_2)
- net SDI: now also J4.3 (Pin_3)
- net SDO: now also J4.4 (Pin_4)
- net SOA: now also J4.6 (Pin_6)
- net SOB: now also J4.7 (Pin_7)
- net SOC: now also J4.8 (Pin_8)
- net VCC: now also C7.1, C_SW1.2, C_VM1.1, R3.1, U1.47 (VIN), U1.6 (VM), C10.1, C9.1, J2.2 (Pin_2); no longer 27uH1.1, C8.1, R1.1, R4.1, R5.1
- net VDRAIN: now also C1.1, C2.1, C3.1; no longer C7.1, C_SW1.2, C_VM1.1, R3.1, U1.47 (VIN), U1.6 (VM)
- net nFAULT: now also J4.5 (Pin_5)
- net nSCS: now also J4.1 (Pin_1)
- new net VAA: 27uH1.1, C8.1, R1.1, R4.1, R5.1
Other:
- note added: "POWER INPUT"

Commit message: Started routing.
Parts:
- L1: renamed from 27uH1; value L -> 27uH
Other:
- moved on the sheet: J4
Changed lines of the file:
@@
 Connection ~ 3450 5700
 $Comp
-L Device:L 27uH1
+L Device:L L1
 U 1 1 5D680E8A
 P 4250 5700
-F 0 "27uH1" V 4100 5700 50  0000 C CNN
-F 1 "L" V 4200 5700 50  0000 C CNN
+F 0 "L1" V 4100 5700 50  0000 C CNN
+F 1 "27uH" V 4200 5700 50  0000 C CNN
 F 2 "Inductor_SMD:L_1210_3225Metric" H 4250 5700 50  0001 C CNN
 F 3 "~" H 4250 5700 50  0001 C CNN
@@
 	1    0    0    -1
 $EndComp
-Text GLabel 4600 2050 0    50   Input ~ 0
+Text GLabel 4600 2100 0    50   Input ~ 0
 SOA
-Text GLabel 4600 2150 0    50   Input ~ 0
+Text GLabel 4600 2200 0    50   Input ~ 0
 SOB
-Text GLabel 4600 2250 0    50   Input ~ 0
+Text GLabel 4600 2300 0    50   Input ~ 0
 SOC
 Text GLabel 4600 1250 0    50   Input ~ 0
@@
 Text GLabel 4600 750  0    50   Input ~ 0
 INLC
-Text GLabel 4600 1850 0    50   Input ~ 0
+Text GLabel 4600 1900 0    50   Input ~ 0
 SDO
-Text GLabel 4600 1750 0    50   Input ~ 0
+Text GLabel 4600 1800 0    50   Input ~ 0
 SDI
-Text GLabel 4600 1650 0    50   Input ~ 0
+Text GLabel 4600 1700 0    50   Input ~ 0
 SCLK
 Text GLabel 4600 1450 0    50   Input ~ 0
@@
 	4600 1450 4700 1450
 Wire Wire Line
-	4600 1550 4700 1550
-Wire Wire Line
-	4600 1650 4700 1650
-Wire Wire Line
-	4600 1750 4700 1750
-Wire Wire Line
-	4600 1850 4700 1850
-Wire Wire Line
-	4600 1950 4700 1950
-Wire Wire Line
-	4600 2050 4700 2050
-Text GLabel 4600 1550 0    50   Input ~ 0
+	4600 1600 4700 1600
+Wire Wire Line
+	4600 1700 4700 1700
+Wire Wire Line
+	4600 1800 4700 1800
+Wire Wire Line
+	4600 1900 4700 1900
+Wire Wire Line
+	4600 2000 4700 2000
+Wire Wire Line
+	4600 2100 4700 2100
+Text GLabel 4600 1600 0    50   Input ~ 0
 nSCS
-Text GLabel 4600 1950 0    50   Input ~ 0
+Text GLabel 4600 2000 0    50   Input ~ 0
 nFAULT
 Wire Wire Line
-	4600 2150 4700 2150
-Wire Wire Line
-	4600 2250 4700 2250
+	4600 2200 4700 2200
+Wire Wire Line
+	4600 2300 4700 2300
 Text GLabel 4600 1350 0    50   Input ~ 0
 DVDD
@@
 L Connector:Conn_01x08_Female J4
 U 1 1 5D68CC07
-P 4900 1850
-F 0 "J4" H 4928 1826 50  0000 L CNN
-F 1 "Pinouts" H 4928 1735 50  0000 L CNN
-F 2 "Connector_PinSocket_2.54mm:PinSocket_1x08_P2.54mm_Vertical" H 4900 1850 50  0001 C CNN
-F 3 "~" H 4900 1850 50  0001 C CNN
-	1    4900 1850
-	1    0    0    -1
-$EndComp
+P 4900 1900
+F 0 "J4" H 4928 1876 50  0000 L CNN
+F 1 "Pinouts" H 4928 1785 50  0000 L CNN
+F 2 "Connector_PinSocket_2.54mm:PinSocket_1x08_P2.54mm_Vertical" H 4900 1900 50  0001 C CNN
+F 3 "~" H 4900 1900 50  0001 C CNN
+	1    4900 1900
+	1    0    0    -1
+$EndComp

Commit message: Still routing.
Connections:
- net VDRAIN is gone; now on net VCC: C1.1, C2.1, C3.1, Q1.1 (D), Q3.1 (D), Q5.1 (D), U1.7 (VDRAIN)
- net VAA: now also C6.1, U1.26 (VREF)
- net VCC: no longer C6.1, U1.26 (VREF)
Changed lines of the file:
@@
 Wire Wire Line
 	8000 3550 8000 3650
-Text GLabel 5600 2600 1    50   Input ~ 0
-VM
-Text GLabel 6800 2600 1    50   Input ~ 0
-VM
-Text GLabel 8000 2600 1    50   Input ~ 0
-VM
 Wire Wire Line
 	6800 2600 6800 2750
@@
 $EndComp
 $Comp
-L power:VCC #PWR05
+L power:VAA #PWR05
 U 1 1 5D62009C
 P 3600 2800
 F 0 "#PWR05" H 3600 2650 50  0001 C CNN
-F 1 "VCC" H 3617 2973 50  0000 C CNN
+F 1 "VAA" H 3617 2973 50  0000 C CNN
 F 2 "" H 3600 2800 50  0001 C CNN
 F 3 "" H 3600 2800 50  0001 C CNN
@@
 	1    0    0    -1
 $EndComp
+$Comp
+L power:VCC #PWR?
+U 1 1 5D6883AB
+P 5600 2600
+F 0 "#PWR?" H 5600 2450 50  0001 C CNN
+F 1 "VCC" H 5617 2773 50  0000 C CNN
+F 2 "" H 5600 2600 50  0001 C CNN
+F 3 "" H 5600 2600 50  0001 C CNN
+	1    5600 2600
+	1    0    0    -1
+$EndComp
+$Comp
+L power:VCC #PWR?
+U 1 1 5D688401
+P 6800 2600
+F 0 "#PWR?" H 6800 2450 50  0001 C CNN
+F 1 "VCC" H 6817 2773 50  0000 C CNN
+F 2 "" H 6800 2600 50  0001 C CNN
+F 3 "" H 6800 2600 50  0001 C CNN
+	1    6800 2600
+	1    0    0    -1
+$EndComp
+$Comp
+L power:VCC #PWR?
+U 1 1 5D68851C
+P 8000 2600
+F 0 "#PWR?" H 8000 2450 50  0001 C CNN
+F 1 "VCC" H 8017 2773 50  0000 C CNN
+F 2 "" H 8000 2600 50  0001 C CNN
+F 3 "" H 8000 2600 50  0001 C CNN
+	1    8000 2600
+	1    0    0    -1
+$EndComp

Commit message: Finished pcb.
Other:
- moved on the sheet: C10, C9, J2, J3, J4

Commit message: Finished board.
Parts:
- U1: footprint Package_DFN_QFN:Texas_S-PVQFN-N48_EP5.15x5.15mm_ThermalVias -> actuator:Texas_S-PVQFN-N48_EP5.15x5.15mm_ThermalVias
Changed lines of the file:
@@
 F 0 "U1" H 2700 5225 50  0000 C CNN
 F 1 "drv8323rs" H 2700 5134 50  0000 C CNN
-F 2 "Package_DFN_QFN:Texas_S-PVQFN-N48_EP5.15x5.15mm_ThermalVias" H 2700 3850 50  0001 C CNN
+F 2 "actuator:Texas_S-PVQFN-N48_EP5.15x5.15mm_ThermalVias" H 2700 3850 50  0001 C CNN
 F 3 "" H 2700 3850 50  0001 C CNN
 	1    2700 3850
@@
 $EndComp
 $Comp
-L power:VCC #PWR?
+L power:VCC #PWR0107
 U 1 1 5D6883AB
 P 5600 2600
-F 0 "#PWR?" H 5600 2450 50  0001 C CNN
+F 0 "#PWR0107" H 5600 2450 50  0001 C CNN
 F 1 "VCC" H 5617 2773 50  0000 C CNN
 F 2 "" H 5600 2600 50  0001 C CNN
@@
 $EndComp
 $Comp
-L power:VCC #PWR?
+L power:VCC #PWR0108
 U 1 1 5D688401
 P 6800 2600
-F 0 "#PWR?" H 6800 2450 50  0001 C CNN
+F 0 "#PWR0108" H 6800 2450 50  0001 C CNN
 F 1 "VCC" H 6817 2773 50  0000 C CNN
 F 2 "" H 6800 2600 50  0001 C CNN
@@
 $EndComp
 $Comp
-L power:VCC #PWR?
+L power:VCC #PWR0109
 U 1 1 5D68851C
 P 8000 2600
-F 0 "#PWR?" H 8000 2450 50  0001 C CNN
+F 0 "#PWR0109" H 8000 2450 50  0001 C CNN
 F 1 "VCC" H 8017 2773 50  0000 C CNN
 F 2 "" H 8000 2600 50  0001 C CNN

Commit message: Updated board.
Parts:
- C1, C2, C3, C7, C8: footprint Capacitor_SMD:C_0603_1608Metric -> Capacitor_SMD:C_1206_3216Metric
- C10, C9: footprint Capacitor_SMD:C_0603_1608Metric -> Capacitor_SMD:CP_Elec_6.3x5.4
- L1: footprint Inductor_SMD:L_1210_3225Metric -> Inductor_THT:L_Radial_D7.8mm_P5.00mm_Fastron_07HCP
- R2: footprint Resistor_SMD:R_0603_1608Metric_Pad1.05x0.95mm_HandSolder -> Resistor_SMD:R_0402_1005Metric
- R6, R7, R8: footprint Resistor_SMD:R_1210_3225Metric -> Resistor_SMD:R_2512_6332Metric
Changed lines of the file:
@@
 F 0 "R6" H 5670 4646 50  0000 L CNN
 F 1 "1m" H 5670 4555 50  0000 L CNN
-F 2 "Resistor_SMD:R_1210_3225Metric" V 5530 4600 50  0001 C CNN
+F 2 "Resistor_SMD:R_2512_6332Metric" V 5530 4600 50  0001 C CNN
 F 3 "~" H 5600 4600 50  0001 C CNN
 	1    5600 4600
@@
 F 0 "R7" H 6870 4646 50  0000 L CNN
 F 1 "1m" H 6870 4555 50  0000 L CNN
-F 2 "Resistor_SMD:R_1210_3225Metric" V 6730 4600 50  0001 C CNN
+F 2 "Resistor_SMD:R_2512_6332Metric" V 6730 4600 50  0001 C CNN
 F 3 "~" H 6800 4600 50  0001 C CNN
 	1    6800 4600
@@
 F 0 "R8" H 8070 4646 50  0000 L CNN
 F 1 "1m" H 8070 4555 50  0000 L CNN
-F 2 "Resistor_SMD:R_1210_3225Metric" V 7930 4600 50  0001 C CNN
+F 2 "Resistor_SMD:R_2512_6332Metric" V 7930 4600 50  0001 C CNN
 F 3 "~" H 8000 4600 50  0001 C CNN
 	1    8000 4600
@@
 F 0 "R2" H 1109 2896 50  0000 L CNN
 F 1 "8.45k" H 1109 2805 50  0000 L CNN
-F 2 "Resistor_SMD:R_0603_1608Metric_Pad1.05x0.95mm_HandSolder" H 1050 2850 50  0001 C CNN
+F 2 "Resistor_SMD:R_0402_1005Metric" H 1050 2850 50  0001 C CNN
 F 3 "~" H 1050 2850 50  0001 C CNN
 	1    1050 2850
@@
 F 0 "L1" V 4100 5700 50  0000 C CNN
 F 1 "27uH" V 4200 5700 50  0000 C CNN
-F 2 "Inductor_SMD:L_1210_3225Metric" H 4250 5700 50  0001 C CNN
+F 2 "Inductor_THT:L_Radial_D7.8mm_P5.00mm_Fastron_07HCP" H 4250 5700 50  0001 C CNN
 F 3 "~" H 4250 5700 50  0001 C CNN
 	1    4250 5700
@@
 F 0 "C8" H 4642 5846 50  0000 L CNN
 F 1 "10uF" H 4642 5755 50  0000 L CNN
-F 2 "Capacitor_SMD:C_0603_1608Metric" H 4550 5800 50  0001 C CNN
+F 2 "Capacitor_SMD:C_1206_3216Metric" H 4550 5800 50  0001 C CNN
 F 3 "~" H 4550 5800 50  0001 C CNN
 	1    4550 5800
@@
 F 0 "C7" H 3792 6296 50  0000 L CNN
 F 1 "10uF" H 3792 6205 50  0000 L CNN
-F 2 "Capacitor_SMD:C_0603_1608Metric" H 3700 6250 50  0001 C CNN
+F 2 "Capacitor_SMD:C_1206_3216Metric" H 3700 6250 50  0001 C CNN
 F 3 "~" H 3700 6250 50  0001 C CNN
 	1    3700 6250
@@
 F 0 "C10" H 3188 1596 50  0000 L CNN
 F 1 "10uF" H 3188 1505 50  0000 L CNN
-F 2 "Capacitor_SMD:C_0603_1608Metric" H 3100 1550 50  0001 C CNN
+F 2 "Capacitor_SMD:CP_Elec_6.3x5.4" H 3100 1550 50  0001 C CNN
 F 3 "~" H 3100 1550 50  0001 C CNN
 	1    3100 1550
@@
 F 0 "C9" H 2788 1596 50  0000 L CNN
 F 1 "10uF" H 2788 1505 50  0000 L CNN
-F 2 "Capacitor_SMD:C_0603_1608Metric" H 2700 1550 50  0001 C CNN
+F 2 "Capacitor_SMD:CP_Elec_6.3x5.4" H 2700 1550 50  0001 C CNN
 F 3 "~" H 2700 1550 50  0001 C CNN
 	1    2700 1550
@@
 F 0 "C1" H 5892 2896 50  0000 L CNN
 F 1 "10uF" H 5892 2805 50  0000 L CNN
-F 2 "Capacitor_SMD:C_0603_1608Metric" H 5800 2850 50  0001 C CNN
+F 2 "Capacitor_SMD:C_1206_3216Metric" H 5800 2850 50  0001 C CNN
 F 3 "~" H 5800 2850 50  0001 C CNN
 	1    5800 2850
@@
 F 0 "C2" H 7092 2896 50  0000 L CNN
 F 1 "10uF" H 7092 2805 50  0000 L CNN
-F 2 "Capacitor_SMD:C_0603_1608Metric" H 7000 2850 50  0001 C CNN
+F 2 "Capacitor_SMD:C_1206_3216Metric" H 7000 2850 50  0001 C CNN
 F 3 "~" H 7000 2850 50  0001 C CNN
 	1    7000 2850
@@
 F 0 "C3" H 8292 2896 50  0000 L CNN
 F 1 "10uF" H 8292 2805 50  0000 L CNN
-F 2 "Capacitor_SMD:C_0603_1608Metric" H 8200 2850 50  0001 C CNN
+F 2 "Capacitor_SMD:C_1206_3216Metric" H 8200 2850 50  0001 C CNN
 F 3 "~" H 8200 2850 50  0001 C CNN
 	1    8200 2850
