File: electronics/jointController/jointController/MA702.sch (KiCad schematic (older format))
At the start: 2 parts

Commit message: Almost done with jointControllerV1
Parts:
- C27: renamed from C?; footprint (none) -> Capacitor_SMD:C_0603_1608Metric_Pad1.05x0.95mm_HandSolder
- U5: renamed from U?; value MA703 -> MA702; footprint (none) -> Package_DFN_QFN:QFN-16-1EP_3x3mm_P0.5mm_EP1.8x1.8mm
Connections:
- net ENC_SDI renamed ENC_MOSI
- net ENC_SDO renamed ENC_MISO
Changed lines of the file:
@@
 $EndDescr
 $Comp
-L jointController:MA703 U?
+L jointController:MA703 U5
 U 1 1 5E579108
 P 5850 4000
-F 0 "U?" H 5450 4550 50  0000 R CNN
-F 1 "MA703" H 6350 4550 50  0000 R CNN
-F 2 "" H 6650 4450 50  0001 C CNN
+F 0 "U5" H 5450 4550 50  0000 R CNN
+F 1 "MA702" H 6350 4550 50  0000 R CNN
+F 2 "Package_DFN_QFN:QFN-16-1EP_3x3mm_P0.5mm_EP1.8x1.8mm" H 6650 4450 50  0001 C CNN
 F 3 "" H 6650 4450 50  0001 C CNN
 	1    5850 4000
@@
 $EndComp
 $Comp
-L Device:C_Small C?
+L Device:C_Small C27
 U 1 1 5E5792AC
 P 5000 4000
-F 0 "C?" H 5092 4046 50  0000 L CNN
+F 0 "C27" H 5092 4046 50  0000 L CNN
 F 1 "1uF" H 5092 3955 50  0000 L CNN
-F 2 "" H 5000 4000 50  0001 C CNN
+F 2 "Capacitor_SMD:C_0603_1608Metric_Pad1.05x0.95mm_HandSolder" H 5000 4000 50  0001 C CNN
 F 3 "~" H 5000 4000 50  0001 C CNN
 	1    5000 4000
@@
 	5000 4100 5250 4100
 $Comp
-L power:+3.3V #PWR?
+L power:+3.3V #PWR058
 U 1 1 5E579308
 P 5000 3450
-F 0 "#PWR?" H 5000 3300 50  0001 C CNN
+F 0 "#PWR058" H 5000 3300 50  0001 C CNN
 F 1 "+3.3V" H 5015 3623 50  0000 C CNN
 F 2 "" H 5000 3450 50  0001 C CNN
@@
 $EndComp
 $Comp
-L power:GND #PWR?
+L power:GND #PWR059
 U 1 1 5E579343
 P 5000 4650
-F 0 "#PWR?" H 5000 4400 50  0001 C CNN
+F 0 "#PWR059" H 5000 4400 50  0001 C CNN
 F 1 "GND" H 5005 4477 50  0000 C CNN
 F 2 "" H 5000 4650 50  0001 C CNN
@@
 Connection ~ 5000 3900
 Text GLabel 6550 3700 2    50   Input ~ 0
-ENC_SDO
+ENC_MISO
 Text GLabel 6550 3800 2    50   Input ~ 0
-ENC_SDI
+ENC_MOSI
 Text GLabel 6550 3900 2    50   Input ~ 0
 ENC_SCLK
@@
 NoConn ~ 6050 4600
 $Comp
-L power:GND #PWR?
+L power:GND #PWR060
 U 1 1 5E579FD7
 P 5650 4650
-F 0 "#PWR?" H 5650 4400 50  0001 C CNN
+F 0 "#PWR060" H 5650 4400 50  0001 C CNN
 F 1 "GND" H 5655 4477 50  0000 C CNN
 F 2 "" H 5650 4650 50  0001 C CNN
@@
 $EndComp
 $Comp
-L power:GND #PWR?
+L power:GND #PWR061
 U 1 1 5E579FFD
 P 5850 4650
-F 0 "#PWR?" H 5850 4400 50  0001 C CNN
+F 0 "#PWR061" H 5850 4400 50  0001 C CNN
 F 1 "GND" H 5855 4477 50  0000 C CNN
 F 2 "" H 5850 4650 50  0001 C CNN
