File: electronics/jointController/jointController/MCP2562.sch (KiCad schematic (older format))
At the start: 4 parts

Commit message: Almost done with jointControllerV1
Parts:
- C25, C26: renamed from C?; footprint (none) -> Capacitor_SMD:C_0603_1608Metric_Pad1.05x0.95mm_HandSolder
- R9: renamed from R?; footprint (none) -> Resistor_SMD:R_0603_1608Metric_Pad1.05x0.95mm_HandSolder
- gave numbers to parts that had none: 1
Changed lines of the file:
@@
 $EndDescr
 $Comp
-L Interface_CAN_LIN:MCP2562-E-MF U?
+L Interface_CAN_LIN:MCP2562-E-MF U4
 U 1 1 5E5788A7
 P 5800 3950
-F 0 "U?" H 5500 4300 50  0000 C CNN
+F 0 "U4" H 5500 4300 50  0000 C CNN
 F 1 "MCP2562-E-MF" H 6150 4300 50  0000 C CNN
 F 2 "Package_DFN_QFN:DFN-8-1EP_3x3mm_P0.65mm_EP1.55x2.4mm" H 5800 3450 50  0001 C CIN
@@
 $EndComp
 $Comp
-L power:+5V #PWR?
+L power:+5V #PWR055
 U 1 1 5E5788AE
 P 5800 3050
-F 0 "#PWR?" H 5800 2900 50  0001 C CNN
+F 0 "#PWR055" H 5800 2900 50  0001 C CNN
 F 1 "+5V" H 5815 3223 50  0000 C CNN
 F 2 "" H 5800 3050 50  0001 C CNN
@@
 $EndComp
 $Comp
-L power:GND #PWR?
+L power:GND #PWR056
 U 1 1 5E5788B4
 P 5800 4350
-F 0 "#PWR?" H 5800 4100 50  0001 C CNN
+F 0 "#PWR056" H 5800 4100 50  0001 C CNN
 F 1 "GND" H 5805 4177 50  0000 C CNN
 F 2 "" H 5800 4350 50  0001 C CNN
@@
 NoConn ~ 5700 4350
 $Comp
-L Device:C_Small C?
+L Device:C_Small C26
 U 1 1 5E5788BF
 P 5950 3200
-F 0 "C?" H 6042 3246 50  0000 L CNN
+F 0 "C26" H 6042 3246 50  0000 L CNN
 F 1 "0.1uF" H 6042 3155 50  0000 L CNN
-F 2 "" H 5950 3200 50  0001 C CNN
+F 2 "Capacitor_SMD:C_0603_1608Metric_Pad1.05x0.95mm_HandSolder" H 5950 3200 50  0001 C CNN
 F 3 "~" H 5950 3200 50  0001 C CNN
 	1    5950 3200
@@
 $EndComp
 $Comp
-L power:GND #PWR?
+L power:GND #PWR057
 U 1 1 5E5788C6
 P 5950 3300
-F 0 "#PWR?" H 5950 3050 50  0001 C CNN
+F 0 "#PWR057" H 5950 3050 50  0001 C CNN
 F 1 "GND" H 5950 3150 50  0000 C CNN
 F 2 "" H 5950 3300 50  0001 C CNN
@@
 STBY
 $Comp
-L power:+3.3V #PWR?
+L power:+3.3V #PWR053
 U 1 1 5E5788D1
 P 4650 4000
-F 0 "#PWR?" H 4650 3850 50  0001 C CNN
+F 0 "#PWR053" H 4650 3850 50  0001 C CNN
 F 1 "+3.3V" H 4665 4173 50  0000 C CNN
 F 2 "" H 4650 4000 50  0001 C CNN
@@
 $EndComp
 $Comp
-L Device:C_Small C?
+L Device:C_Small C25
 U 1 1 5E5788D7
 P 4650 4200
-F 0 "C?" H 4742 4246 50  0000 L CNN
+F 0 "C25" H 4742 4246 50  0000 L CNN
 F 1 "0.1uF" H 4742 4155 50  0000 L CNN
-F 2 "" H 4650 4200 50  0001 C CNN
+F 2 "Capacitor_SMD:C_0603_1608Metric_Pad1.05x0.95mm_HandSolder" H 4650 4200 50  0001 C CNN
 F 3 "~" H 4650 4200 50  0001 C CNN
 	1    4650 4200
@@
 $EndComp
 $Comp
-L power:GND #PWR?
+L power:GND #PWR054
 U 1 1 5E5788DE
 P 4650 4350
-F 0 "#PWR?" H 4650 4100 50  0001 C CNN
+F 0 "#PWR054" H 4650 4100 50  0001 C CNN
 F 1 "GND" H 4655 4177 50  0000 C CNN
 F 2 "" H 4650 4350 50  0001 C CNN
@@
 	5250 4150 5300 4150
 $Comp
-L Device:R_Small R?
+L Device:R_Small R9
 U 1 1 5E5788EC
 P 6500 3950
-F 0 "R?" H 6559 3996 50  0000 L CNN
+F 0 "R9" H 6559 3996 50  0000 L CNN
 F 1 "120" H 6559 3905 50  0000 L CNN
-F 2 "" H 6500 3950 50  0001 C CNN
+F 2 "Resistor_SMD:R_0603_1608Metric_Pad1.05x0.95mm_HandSolder" H 6500 3950 50  0001 C CNN
 F 3 "~" H 6500 3950 50  0001 C CNN
 	1    6500 3950
