File: electronics/jointController/jointController/drv8323.sch (KiCad schematic (older format))
At the start: 16 parts

Commit message: Almost done with jointControllerV1
Parts:
- removed R?: 100k, symbol Device:R_Small
- C10: renamed from C?; footprint (none) -> Capacitor_SMD:C_0603_1608Metric_Pad1.05x0.95mm_HandSolder
- C11: renamed from C?; footprint (none) -> Capacitor_SMD:C_1206_3216Metric_Pad1.42x1.75mm_HandSolder
- C12: renamed from C?; value 10uF -> 22uF; footprint (none) -> Capacitor_SMD:C_0603_1608Metric_Pad1.05x0.95mm_HandSolder
- C_SW1: renamed from C_SW?; footprint (none) -> Capacitor_SMD:C_0603_1608Metric_Pad1.05x0.95mm_HandSolder
- C_VCP1: renamed from C_VCP?; footprint (none) -> Capacitor_SMD:C_0603_1608Metric_Pad1.05x0.95mm_HandSolder
- C_VDD1: renamed from C_VDD?; footprint (none) -> Capacitor_SMD:C_0603_1608Metric_Pad1.05x0.95mm_HandSolder
- C_VM1: renamed from C_VM?; footprint (none) -> Capacitor_SMD:C_0603_1608Metric_Pad1.05x0.95mm_HandSolder
- C_VREF1: renamed from C_VREF?; footprint (none) -> Capacitor_SMD:C_0603_1608Metric_Pad1.05x0.95mm_HandSolder
- D1: renamed from D?; footprint (none) -> Diode_SMD:D_SOD-123F
- L1: renamed from L?; value 27uH -> 22uH; footprint (none) -> jointController:NRH3012T220MN
- R_FB1: renamed from R_FB?; value 28k -> 54.9k; footprint (none) -> Resistor_SMD:R_0603_1608Metric_Pad1.05x0.95mm_HandSolder
- R_FB2: renamed from R_FB?; value 8.45k -> 10k; footprint (none) -> Resistor_SMD:R_0603_1608Metric_Pad1.05x0.95mm_HandSolder
- R_PU1: renamed from R_PU?; footprint (none) -> Resistor_SMD:R_0603_1608Metric_Pad1.05x0.95mm_HandSolder
- R_PU2: renamed from R_PU?; value R_Small -> 10k; footprint (none) -> Resistor_SMD:R_0603_1608Metric_Pad1.05x0.95mm_HandSolder
- U2: renamed from U?; footprint (none) -> jointController:VQFN-48-7x7-P0.5
Connections:
- net INLB is gone; now on net PWM_EN: U2.40 (INLB)
- net INLC is gone; now on net PWM_EN: U2.42 (INLC)
- net +3V3: no longer C12.1, L1.2, R_FB1.1
- net CAL: no longer names the net of U2.34 (CAL)
- net DRV_SDI renamed DRV_MOSI
- net DRV_SDO renamed DRV_MISO
- net DVDD: no longer names the net of C_VDD1.2, U2.36 (DVDD)
- net INLA renamed PWM_EN
- net SNC: no longer names the net of U2.22 (SNC)
- net SOC: no longer names the net of U2.23 (SOC)
- net SPC: no longer names the net of U2.21 (SPC)
- net VDRAIN renamed V_DRAIN
- new net +5V: C12.1, L1.2, R_FB1.1
- no-connect marks 1 -> 6
