File: electronics/jointController/jointController/dsPIC33CK256MP508.sch (KiCad schematic (older format))
At the start: 23 parts

Commit message: Almost done with jointControllerV1
Parts:
- removed R? (x3): 75, symbol Device:R_Small
- added TP1: DACOUT1, Connector_PinHeader_1.00mm:PinHeader_1x01_P1.00mm_Vertical, symbol Connector:TestPoint
- C13, C14, C15, C16, C17, C18, C19, C20, C21, C22, C23, C24: renamed from C?; footprint (none) -> Capacitor_SMD:C_0603_1608Metric_Pad1.05x0.95mm_HandSolder
- L2: renamed from L?; footprint (none) -> Inductor_SMD:L_0603_1608Metric_Pad1.05x0.95mm_HandSolder
- R3, R4, R5, R6, R7, R8: renamed from R?; footprint (none) -> Resistor_SMD:R_0603_1608Metric_Pad1.05x0.95mm_HandSolder
- U3: renamed from U?; footprint (none) -> Package_QFP:TQFP-80_12x12mm_P0.5mm
Connections:
- net PWM_EN: now reaches U3.2 (RE0)
- net at U3.21 (RA3): now also TP1.1
- net PWRGD: now reaches C14.1, R3.1, R4.2, U3.9 (nMCLR)
- net DRV_SDI renamed DRV_MOSI
- net DRV_SDO renamed DRV_MISO
- net ENC_SDI renamed ENC_MOSI
- net ENC_SDO renamed ENC_MISO
- no-connect marks 0 -> 45
Other:
- moved on the sheet: C14, R3, R4
