File: electronics/jointController/jointController/three_phase_inverter.sch (KiCad schematic (older format))
At the start: 12 parts

Commit message: Almost done with jointControllerV1
Parts:
- removed R?: 1m, symbol Device:R_Small
- C7, C8, C9: renamed from C?; footprint (none) -> Capacitor_SMD:C_1206_3216Metric_Pad1.42x1.75mm_HandSolder
- Q1, Q2, Q3, Q4, Q5, Q6: renamed from Q?; footprint (none) -> jointController:8-SOFL
- R1, R2: renamed from R?; footprint (none) -> Resistor_SMD:R_2512_6332Metric_Pad1.52x3.35mm_HandSolder
Connections:
- net SPC is gone; now on net GND: Q6.3 (S)
Changed lines of the file:
@@
 $EndDescr
 $Comp
-L Device:Q_NMOS_DGS Q?
+L Device:Q_NMOS_DGS Q1
 U 1 1 5E5F911B
 P 4200 3300
-F 0 "Q?" H 4406 3346 50  0000 L CNN
+F 0 "Q1" H 4406 3346 50  0000 L CNN
 F 1 "NTMFS4935NT1G" H 4406 3255 50  0000 L CNN
-F 2 "" H 4400 3400 50  0001 C CNN
+F 2 "jointController:8-SOFL" H 4400 3400 50  0001 C CNN
 F 3 "~" H 4200 3300 50  0001 C CNN
 	1    4200 3300
@@
 $EndComp
 $Comp
-L Device:Q_NMOS_DGS Q?
+L Device:Q_NMOS_DGS Q2
 U 1 1 5E5F9122
 P 4200 4000
-F 0 "Q?" H 4406 4046 50  0000 L CNN
+F 0 "Q2" H 4406 4046 50  0000 L CNN
 F 1 "NTMFS4935NT1G" H 4406 3955 50  0000 L CNN
-F 2 "" H 4400 4100 50  0001 C CNN
+F 2 "jointController:8-SOFL" H 4400 4100 50  0001 C CNN
 F 3 "~" H 4200 4000 50  0001 C CNN
 	1    4200 4000
@@
 $EndComp
 $Comp
-L Device:C_Small C?
+L Device:C_Small C7
 U 1 1 5E5F9129
 P 4600 2900
-F 0 "C?" H 4692 2946 50  0000 L CNN
+F 0 "C7" H 4692 2946 50  0000 L CNN
 F 1 "10uF" H 4692 2855 50  0000 L CNN
-F 2 "" H 4600 2900 50  0001 C CNN
+F 2 "Capacitor_SMD:C_1206_3216Metric_Pad1.42x1.75mm_HandSolder" H 4600 2900 50  0001 C CNN
 F 3 "~" H 4600 2900 50  0001 C CNN
 	1    4600 2900
@@
 $EndComp
 $Comp
-L power:GND #PWR?
+L power:GND #PWR016
 U 1 1 5E5F9130
 P 4600 3000
-F 0 "#PWR?" H 4600 2750 50  0001 C CNN
+F 0 "#PWR016" H 4600 2750 50  0001 C CNN
 F 1 "GND" H 4605 2827 50  0000 C CNN
 F 2 "" H 4600 3000 50  0001 C CNN
@@
 $EndComp
 $Comp
-L power:VCC #PWR?
+L power:VCC #PWR014
 U 1 1 5E5F9136
 P 4300 2750
-F 0 "#PWR?" H 4300 2600 50  0001 C CNN
+F 0 "#PWR014" H 4300 2600 50  0001 C CNN
 F 1 "VCC" H 4317 2923 50  0000 C CNN
 F 2 "" H 4300 2750 50  0001 C CNN
@@
 GLA
 $Comp
-L Device:R_Small R?
+L Device:R_Small R1
 U 1 1 5E5F913F
 P 4300 4500
-F 0 "R?" H 4359 4546 50  0000 L CNN
+F 0 "R1" H 4359 4546 50  0000 L CNN
 F 1 "1m" H 4359 4455 50  0000 L CNN
-F 2 "" H 4300 4500 50  0001 C CNN
+F 2 "Resistor_SMD:R_2512_6332Metric_Pad1.52x3.35mm_HandSolder" H 4300 4500 50  0001 C CNN
 F 3 "~" H 4300 4500 50  0001 C CNN
 	1    4300 4500
@@
 SNA
 $Comp
-L power:GND #PWR?
+L power:GND #PWR015
 U 1 1 5E5F9148
 P 4300 4800
-F 0 "#PWR?" H 4300 4550 50  0001 C CNN
+F 0 "#PWR015" H 4300 4550 50  0001 C CNN
 F 1 "GND" H 4305 4627 50  0000 C CNN
 F 2 "" H 4300 4800 50  0001 C CNN
@@
 	4300 4700 4300 4800
 $Comp
-L Device:Q_NMOS_DGS Q?
+L Device:Q_NMOS_DGS Q3
 U 1 1 5E5F9162
 P 5650 3300
-F 0 "Q?" H 5856 3346 50  0000 L CNN
+F 0 "Q3" H 5856 3346 50  0000 L CNN
 F 1 "NTMFS4935NT1G" H 5856 3255 50  0000 L CNN
-F 2 "" H 5850 3400 50  0001 C CNN
+F 2 "jointController:8-SOFL" H 5850 3400 50  0001 C CNN
 F 3 "~" H 5650 3300 50  0001 C CNN
 	1    5650 3300
@@
 $EndComp
 $Comp
-L Device:Q_NMOS_DGS Q?
+L Device:Q_NMOS_DGS Q4
 U 1 1 5E5F9169
 P 5650 4000
-F 0 "Q?" H 5856 4046 50  0000 L CNN
+F 0 "Q4" H 5856 4046 50  0000 L CNN
 F 1 "NTMFS4935NT1G" H 5856 3955 50  0000 L CNN
-F 2 "" H 5850 4100 50  0001 C CNN
+F 2 "jointController:8-SOFL" H 5850 4100 50  0001 C CNN
 F 3 "~" H 5650 4000 50  0001 C CNN
 	1    5650 4000
@@
 $EndComp
 $Comp
-L Device:C_Small C?
+L Device:C_Small C8
 U 1 1 5E5F9170
 P 6050 2900
-F 0 "C?" H 6142 2946 50  0000 L CNN
+F 0 "C8" H 6142 2946 50  0000 L CNN
 F 1 "10uF" H 6142 2855 50  0000 L CNN
-F 2 "" H 6050 2900 50  0001 C CNN
+F 2 "Capacitor_SMD:C_1206_3216Metric_Pad1.42x1.75mm_HandSolder" H 6050 2900 50  0001 C CNN
 F 3 "~" H 6050 2900 50  0001 C CNN
 	1    6050 2900
@@
 $EndComp
 $Comp
-L power:GND #PWR?
+L power:GND #PWR019
 U 1 1 5E5F9177
 P 6050 3000
-F 0 "#PWR?" H 6050 2750 50  0001 C CNN
+F 0 "#PWR019" H 6050 2750 50  0001 C CNN
 F 1 "GND" H 6055 2827 50  0000 C CNN
 F 2 "" H 6050 3000 50  0001 C CNN
@@
 $EndComp
 $Comp
-L power:VCC #PWR?
+L power:VCC #PWR017
 U 1 1 5E5F917D
 P 5750 2750
-F 0 "#PWR?" H 5750 2600 50  0001 C CNN
+F 0 "#PWR017" H 5750 2600 50  0001 C CNN
 F 1 "VCC" H 5767 2923 50  0000 C CNN
 F 2 "" H 5750 2750 50  0001 C CNN
@@
 GLB
 $Comp
-L Device:R_Small R?
+L Device:R_Small R2
 U 1 1 5E5F9186
 P 5750 4500
-F 0 "R?" H 5809 4546 50  0000 L CNN
+F 0 "R2" H 5809 4546 50  0000 L CNN
 F 1 "1m" H 5809 4455 50  0000 L CNN
-F 2 "" H 5750 4500 50  0001 C CNN
+F 2 "Resistor_SMD:R_2512_6332Metric_Pad1.52x3.35mm_HandSolder" H 5750 4500 50  0001 C CNN
 F 3 "~" H 5750 4500 50  0001 C CNN
 	1    5750 4500
@@
 SNB
 $Comp
-L power:GND #PWR?
+L power:GND #PWR018
 U 1 1 5E5F918F
 P 5750 4800
-F 0 "#PWR?" H 5750 4550 50  0001 C CNN
+F 0 "#PWR018" H 5750 4550 50  0001 C CNN
 F 1 "GND" H 5755 4627 50  0000 C CNN
 F 2 "" H 5750 4800 50  0001 C CNN
@@
 	5750 4700 5750 4800
 $Comp
-L Device:Q_NMOS_DGS Q?
+L Device:Q_NMOS_DGS Q5
 U 1 1 5E5F91A9
 P 7100 3300
-F 0 "Q?" H 7306 3346 50  0000 L CNN
+F 0 "Q5" H 7306 3346 50  0000 L CNN
 F 1 "NTMFS4935NT1G" H 7306 3255 50  0000 L CNN
-F 2 "" H 7300 3400 50  0001 C CNN
+F 2 "jointController:8-SOFL" H 7300 3400 50  0001 C CNN
 F 3 "~" H 7100 3300 50  0001 C CNN
 	1    7100 3300
@@
 $EndComp
 $Comp
-L Device:Q_NMOS_DGS Q?
+L Device:Q_NMOS_DGS Q6
 U 1 1 5E5F91B0
 P 7100 4000
-F 0 "Q?" H 7306 4046 50  0000 L CNN
+F 0 "Q6" H 7306 4046 50  0000 L CNN
 F 1 "NTMFS4935NT1G" H 7306 3955 50  0000 L CNN
-F 2 "" H 7300 4100 50  0001 C CNN
+F 2 "jointController:8-SOFL" H 7300 4100 50  0001 C CNN
 F 3 "~" H 7100 4000 50  0001 C CNN
 	1    7100 4000
@@
 $EndComp
 $Comp
-L Device:C_Small C?
+L Device:C_Small C9
 U 1 1 5E5F91B7
 P 7500 2900
-F 0 "C?" H 7592 2946 50  0000 L CNN
+F 0 "C9" H 7592 2946 50  0000 L CNN
 F 1 "10uF" H 7592 2855 50  0000 L CNN
-F 2 "" H 7500 2900 50  0001 C CNN
+F 2 "Capacitor_SMD:C_1206_3216Metric_Pad1.42x1.75mm_HandSolder" H 7500 2900 50  0001 C CNN
 F 3 "~" H 7500 2900 50  0001 C CNN
 	1    7500 2900
@@
 $EndComp
 $Comp
-L power:GND #PWR?
+L power:GND #PWR022
 U 1 1 5E5F91BE
 P 7500 3000
-F 0 "#PWR?" H 7500 2750 50  0001 C CNN
+F 0 "#PWR022" H 7500 2750 50  0001 C CNN
 F 1 "GND" H 7505 2827 50  0000 C CNN
 F 2 "" H 7500 3000 50  0001 C CNN
@@
 $EndComp
 $Comp
-L power:VCC #PWR?
+L power:VCC #PWR020
 U 1 1 5E5F91C4
 P 7200 2750
-F 0 "#PWR?" H 7200 2600 50  0001 C CNN
+F 0 "#PWR020" H 7200 2600 50  0001 C CNN
 F 1 "VCC" H 7217 2923 50  0000 C CNN
 F 2 "" H 7200 2750 50  0001 C CNN
@@
 GLC
 $Comp
-L Device:R_Small R?
-U 1 1 5E5F91CD
-P 7200 4500
-F 0 "R?" H 7259 4546 50  0000 L CNN
-F 1 "1m" H 7259 4455 50  0000 L CNN
-F 2 "" H 7200 4500 50  0001 C CNN
-F 3 "~" H 7200 4500 50  0001 C CNN
-	1    7200 4500
-	1    0    0    -1
-$EndComp
-Text GLabel 6800 4300 0    50   Input ~ 0
-SPC
-Text GLabel 6800 4700 0    50   Input ~ 0
-SNC
-$Comp
-L power:GND #PWR?
+L power:GND #PWR021
 U 1 1 5E5F91D6
 P 7200 4800
-F 0 "#PWR?" H 7200 4550 50  0001 C CNN
+F 0 "#PWR021" H 7200 4550 50  0001 C CNN
 F 1 "GND" H 7205 4627 50  0000 C CNN
 F 2 "" H 7200 4800 50  0001 C CNN
@@
 Wire Wire Line
 	6800 4000 6900 4000
-Wire Wire Line
-	7200 4200 7200 4300
-Wire Wire Line
-	6800 4300 7200 4300
-Connection ~ 7200 4300
-Wire Wire Line
-	7200 4300 7200 4400
-Wire Wire Line
-	7200 4600 7200 4700
-Wire Wire Line
-	6800 4700 7200 4700
-Connection ~ 7200 4700
-Wire Wire Line
-	7200 4700 7200 4800
 Text GLabel 5500 2800 0    50   Input ~ 0
 V_DRAIN
 Wire Wire Line
 	5500 2800 5750 2800
+Wire Wire Line
+	7200 4200 7200 4800
 $EndSCHEMATC
