File: electronics/jointController/jointController/jointController.kicad_pcb (KiCad board)
At the start: 2 copper layers, 50 x 50 mm, 68 parts, among them J1 PWR_IN, J2 ICSP, J3 CAN, J4 A_OUT, J5 B_OUT, J6 C_OUT, J7 UART1, J8 CAN, Q1 NTMFS4935NT1G, Q2 NTMFS4935NT1G, Q3 NTMFS4935NT1G, Q4 NTMFS4935NT1G, Q5 NTMFS4935NT1G, Q6 NTMFS4935NT1G, U1 MCP1755-3v3, U2 DRV8323RS, U3 dsPIC33CK256MP508, U4 MCP2562-E-MF, U5 MA703

Commit message: jointController V1.0 finished.
Parts:
- J1: footprint Connector_PinHeader_2.54mm:PinHeader_1x02_P2.54mm_Vertical -> Connector_Wire:SolderWirePad_1x02_P5.08mm_Drill1.5mm
- J4, J5, J6: footprint Connector_PinHeader_2.54mm:PinHeader_1x01_P2.54mm_Vertical -> Connector_Wire:SolderWirePad_1x01_Drill1.5mm
- U5: value MA703 -> MA702
- moved J1 1.66 mm to (125.9, 92.1), turned to 270 degrees
- moved C1 0.38 mm to (127.3, 100.5)
- moved C26 0.13 mm to (160.7, 98.3)
Connections:
- U2 pad 49: (no net) -> SNA
Routing:
- net SNA: track 44.2 -> 47.8 mm, vias 28 -> 67
- net +5V: track 65.4 -> 68.4 mm
- net V_DRAIN: vias 12 -> 25
- added copper zone on B.Cu, net A_OUT
- added copper zone on B.Cu, net B_OUT
- added copper zone on B.Cu, net C_OUT
- added copper zone on B.Cu, net V_DRAIN
Other:
- board text added: "jointController v1.0"
