File: electronics/jointController/jointController/jointController.sch (KiCad schematic (older format))
At the start: 8 parts

Commit message: Almost done with jointControllerV1
Parts:
- removed J?: MOTOR_OUT, symbol Connector:Conn_01x03_Female
- added C4: 10uF, Capacitor_SMD:C_1206_3216Metric_Pad1.42x1.75mm_HandSolder, symbol Device:C_Small
- added C5, C6: 10uF, Capacitor_SMD:C_0603_1608Metric_Pad1.05x0.95mm_HandSolder, symbol Device:C_Small
- added J4: A_OUT, Connector_PinHeader_2.54mm:PinHeader_1x01_P2.54mm_Vertical, symbol Connector:Conn_01x01_Female
- added J5: B_OUT, Connector_PinHeader_2.54mm:PinHeader_1x01_P2.54mm_Vertical, symbol Connector:Conn_01x01_Female
- added J6: C_OUT, Connector_PinHeader_2.54mm:PinHeader_1x01_P2.54mm_Vertical, symbol Connector:Conn_01x01_Female
- added J8: CAN, Connector_JST:JST_SH_BM03B-SRSS-TB_1x03-1MP_P1.00mm_Vertical, symbol Connector:Conn_01x03_Female
- added U1: MCP1755-3v3, Package_TO_SOT_SMD:SOT-23-5, symbol jointController:MCP1755-3v3
- C1, C2, C3: renamed from C?; footprint (none) -> Capacitor_SMD:C_1206_3216Metric_Pad1.42x1.75mm_HandSolder; symbol Device:CP_Small -> Device:C_Small
- J1: renamed from J?; footprint (none) -> Connector_PinHeader_2.54mm:PinHeader_1x02_P2.54mm_Vertical
- J2: renamed from J?; footprint (none) -> jointController:PinHeader_1x06_P2.54mm_Vertical_Staggered
- J3, J7: renamed from J?; footprint (none) -> Connector_JST:JST_SH_BM03B-SRSS-TB_1x03-1MP_P1.00mm_Vertical
Connections:
- net +3V3: now also C6.1, U1.5 (VOUT)
- net A_OUT: now also J4.1 (Pin_1)
- net B_OUT: now also J5.1 (Pin_1)
- net CANH: now also J8.1 (Pin_1)
- net CANL: now also J8.2 (Pin_2)
- net C_OUT: now also J6.1 (Pin_1)
- net GND: now also C4.2, C5.2, C6.2, J8.3 (Pin_3), U1.2 (GND)
- net VCC: now also C4.1
- new net +5V: C5.1, U1.1 (VIN), U1.3 (SHDN)
- new net PWRGD: U1.4 (PWRGD)
Other:
- note added: "3.3V Regulator"
- note added: "MOTOR_OUT"
- note removed: "MOTOR OUTPUT"
- moved on the sheet: J2, J3, J7

Commit message: jointController V1.0 finished.
Parts:
- J1: footprint Connector_PinHeader_2.54mm:PinHeader_1x02_P2.54mm_Vertical -> Connector_Wire:SolderWirePad_1x02_P5.08mm_Drill1.5mm
- J4, J5, J6: footprint Connector_PinHeader_2.54mm:PinHeader_1x01_P2.54mm_Vertical -> Connector_Wire:SolderWirePad_1x01_Drill1.5mm
Changed lines of the file:
@@
 F 0 "J1" H 794 925 50  0000 C CNN
 F 1 "PWR_IN" H 794 1016 50  0000 C CNN
-F 2 "Connector_PinHeader_2.54mm:PinHeader_1x02_P2.54mm_Vertical" H 900 1250 50  0001 C CNN
+F 2 "Connector_Wire:SolderWirePad_1x02_P5.08mm_Drill1.5mm" H 900 1250 50  0001 C CNN
 F 3 "~" H 900 1250 50  0001 C CNN
 	1    900  1250
@@
 F 0 "J4" H 8727 3376 50  0000 L CNN
 F 1 "A_OUT" H 8727 3285 50  0000 L CNN
-F 2 "Connector_PinHeader_2.54mm:PinHeader_1x01_P2.54mm_Vertical" H 8700 3350 50  0001 C CNN
+F 2 "Connector_Wire:SolderWirePad_1x01_Drill1.5mm" H 8700 3350 50  0001 C CNN
 F 3 "~" H 8700 3350 50  0001 C CNN
 	1    8700 3350
@@
 F 0 "J5" H 8728 3576 50  0000 L CNN
 F 1 "B_OUT" H 8728 3485 50  0000 L CNN
-F 2 "Connector_PinHeader_2.54mm:PinHeader_1x01_P2.54mm_Vertical" H 8700 3550 50  0001 C CNN
+F 2 "Connector_Wire:SolderWirePad_1x01_Drill1.5mm" H 8700 3550 50  0001 C CNN
 F 3 "~" H 8700 3550 50  0001 C CNN
 	1    8700 3550
@@
 F 0 "J6" H 8728 3776 50  0000 L CNN
 F 1 "C_OUT" H 8728 3685 50  0000 L CNN
-F 2 "Connector_PinHeader_2.54mm:PinHeader_1x01_P2.54mm_Vertical" H 8700 3750 50  0001 C CNN
+F 2 "Connector_Wire:SolderWirePad_1x01_Drill1.5mm" H 8700 3750 50  0001 C CNN
 F 3 "~" H 8700 3750 50  0001 C CNN
 	1    8700 3750
